Commit message: Project: Renamed from ekf_simulator to robotuna_ekf_simulator

File: urdf/Kwad.xacro (robot description, xacro)
@@ -11,6 +11,6 @@
 	<xacro:property name="prop_loc" value="0.15909" />
 <!-- ======================================================== -->
-	<xacro:include filename="$(find ekf_simulator)/urdf/material.xacro" />
-	<xacro:include filename="$(find ekf_simulator)/urdf/Kwad.gazebo" />
+	<xacro:include filename="$(find robotuna_ekf_simulator)/urdf/material.xacro" />
+	<xacro:include filename="$(find robotuna_ekf_simulator)/urdf/Kwad.gazebo" />
 <!-- ======================================================== -->
 	<!-- Define inertial macro -->
@@ -166,5 +166,5 @@
 			<origin xyz="0 0 0" rpy="0 0 0" />
 			<geometry>
-				<mesh filename="package://ekf_simulator/meshes/22V10.dae" scale="0.005 0.005 0.005" />
+				<mesh filename="package://robotuna_ekf_simulator/meshes/22V10.dae" scale="0.005 0.005 0.005" />
 			</geometry>
 		</visual>

Commit message: URDF: Cleared camera view, added IMU, cleaned up unused parts

File: urdf/Kwad.xacro (robot description, xacro)
@@ -24,5 +24,5 @@
 	</xacro:macro>
 <!-- ======================================================== -->
-	<link name="base_link1">
+	<link name="arm_1">
 		<visual>
 			<origin xyz="0 0 0" rpy="0 0 ${pi_value/4}" />
@@ -41,5 +41,5 @@
 	</link>
 <!-- ======================================================== -->
-	<link name="base_link2">
+	<link name="arm_2">
 		<visual>
 			<origin xyz="0 0 0" rpy="0 0 ${-pi_value/4}" />
@@ -77,21 +77,4 @@
 	</link>
 <!-- ======================================================== -->
-	<link name="plate2">
-		<visual>
-			<origin xyz="0 0 0" rpy="0 0 0" />
-			<geometry>
-				<box size="${0.05} ${0.03} ${0.005}" />
-			</geometry>
-			<material name="blue" />
-		</visual>
-		<collision>
-			<origin xyz="0 0 0" rpy="0 0 0" />
-			<geometry>
-				<box size="${0.05} ${0.03} ${0.005}" />
-			</geometry>
-		</collision>
-		<xacro:default_inertial mass="${0.001}" p="${0}" ix_value="${0}" iy_value="${0}" iz_value="${8.1666-7}" />
-	</link>
-<!-- ======================================================== -->
 	<link name="cyl1">
 		<visual>
@@ -162,21 +145,22 @@
 	</link>
 <!-- ======================================================== -->
-	<link name="arduino">
-		<visual>
-			<origin xyz="0 0 0" rpy="0 0 0" />
-			<geometry>
-				<mesh filename="package://robotuna_ekf_simulator/meshes/22V10.dae" scale="0.005 0.005 0.005" />
-			</geometry>
-		</visual>
-		<collision>
-			<origin xyz="0 0 0" rpy="0 0 0" />
-			<geometry>
-				<box size="0.1 0.1 0.001" />
-			</geometry>
-		</collision>
-		<xacro:default_inertial mass="${0.05}" p="${0}" ix_value="${0}" iy_value="${0}" iz_value="${8.33333e-5}" />
-	</link>
-<!-- ======================================================== -->
 	<link name="camera_link">
+		<visual>
+			<origin xyz="0 0 0" rpy="0 0 0" />
+			<geometry>
+				<box size="0.01 0.01 0.01" />
+			</geometry>
+			<material name="red" />
+		</visual>
+		<collision>
+			<origin xyz="0 0 0" rpy="0 0 0" />
+			<geometry>
+				<box size="0.01 0.01 0.01" />
+			</geometry>
+		</collision>
+		<xacro:default_inertial mass="${1e-5}" p="${0}" ix_value="${1e-6}" iy_value="${1e-6}" iz_value="${1e-6}" />
+	</link>
+<!-- ======================================================== -->
+	<link name="imu_link">
 		<visual>
 			<origin xyz="0 0 0" rpy="0 0 0" />
@@ -263,11 +247,11 @@
 	<joint name="base_joint" type="fixed">
 		<parent link="base_link" />
-		<child link="base_link1" />
+		<child link="arm_1" />
 		<origin xyz="0 0 0" rpy="0 0 0" />
   	</joint>
 	<!-- Define the joint between the arms of the frame -->
 	<joint name="center" type="fixed">
-		<parent link="base_link1" />
-		<child link="base_link2" />
+		<parent link="arm_1" />
+		<child link="arm_2" />
 		<origin xyz="0 0 0" rpy="0 0 0"/>
 		<axis xyz="0 0 1" />
@@ -276,5 +260,5 @@
 	<!-- Define joint between prop fr and frame -->
 	<joint name="joint_front_right_prop" type="continuous">
-		<parent link="base_link2" />
+		<parent link="arm_2" />
 		<child link="prop_front_right" />
 		<origin xyz="${prop_loc - 0.01} ${prop_loc - 0.01} 0.021" rpy="0 0 0"/>
@@ -284,5 +268,5 @@
 	<!-- Define joint between prop fl and frame -->
 	<joint name="joint_front_left_prop" type="continuous">
-		<parent link="base_link1" />
+		<parent link="arm_1" />
 		<child link="prop_front_left" />
 		<origin xyz="${-prop_loc + 0.01} ${prop_loc - 0.01} 0.021" rpy="0 0 0" />
@@ -292,5 +276,5 @@
 <!-- Define joint between prop br and frame -->
 	<joint name="joint_back_right_prop" type="continuous">
-		<parent link="base_link1" />
+		<parent link="arm_1" />
 		<child link="prop_back_right" />
 		<origin xyz="${prop_loc - 0.01} ${-prop_loc + 0.01} 0.021" rpy="0 0 0" />
@@ -300,5 +284,5 @@
 <!-- Define joint between prop br and frame -->
 	<joint name="joint_back_left_prop" type="continuous">
-		<parent link="base_link2" />
+		<parent link="arm_2" />
 		<child link="prop_back_left" />
 		<origin xyz="${-prop_loc + 0.01} ${-prop_loc + 0.01} 0.021" rpy="0 0 0" />
@@ -308,5 +292,5 @@
 <!-- Define joint between plate1 and frame -->
 	<joint name="joint_plate1_frame" type="fixed">
-		<parent link="base_link2" />
+		<parent link="arm_2" />
 		<child link="plate1" />
 		<origin xyz="${0} ${0} 0.005" rpy="0 0 0" />
@@ -314,15 +298,7 @@
 	</joint>
 <!-- ======================================================== -->
-<!-- Define joint between plate1 and plate2 -->
-	<joint name="joint_plate2_frame" type="fixed">
-		<parent link="plate1" />
-		<child link="plate2" />
-		<origin xyz="${0} ${0} 0.007" rpy="0 0 0" />
-		<axis xyz="0 0 1" />
-	</joint>
-<!-- ======================================================== -->
 <!-- Define joint between cyl1 and frame -->
 	<joint name="joint_cyl1_frame" type="fixed">
-		<parent link="base_link2" />
+		<parent link="arm_2" />
 		<child link="cyl1" />
 		<origin xyz="${prop_loc - 0.01} ${prop_loc - 0.01} 0.01" rpy="0 0 0" />
@@ -332,5 +308,5 @@
 <!-- Define joint between cyl2 and frame -->
 	<joint name="joint_cyl2_frame" type="fixed">
-		<parent link="base_link2" />
+		<parent link="arm_2" />
 		<child link="cyl2" />
 		<origin xyz="${-prop_loc + 0.01} ${-prop_loc + 0.01} 0.01" rpy="0 0 0" />
@@ -340,5 +316,5 @@
 <!-- Define joint between cyl3 and frame -->
 	<joint name="joint_cyl3_frame" type="fixed">
-		<parent link="base_link1" />
+		<parent link="arm_1" />
 		<child link="cyl3" />
 		<origin xyz="${-prop_loc + 0.01} ${prop_loc - 0.01} 0.01" rpy="0 0 0" />
@@ -348,5 +324,5 @@
 <!-- Define joint between cyl4 and frame -->
 	<joint name="joint_cyl4_frame" type="fixed">
-		<parent link="base_link1" />
+		<parent link="arm_1" />
 		<child link="cyl4" />
 		<origin xyz="${prop_loc - 0.01} ${-prop_loc + 0.01} 0.01" rpy="0 0 0" />
@@ -354,18 +330,17 @@
 	</joint>
 <!-- ======================================================== -->
-<!-- Define joint between Arduino and frame -->
-	<joint name="joint_arduino_frame" type="fixed">
-		<parent link="plate2" />
-		<child link="arduino" />
-		<origin xyz="${0} ${0} 0.005" rpy="0 0 0" />
-		<axis xyz="0 0 1" />
-	</joint>
-<!-- ======================================================== -->
-<!-- Define joint between Arduino and frame -->
+<!-- Define joint between camera and frame -->
 	<joint name="joint_camera_frame" type="fixed">
-		<parent link="plate2" />
+		<parent link="plate1" />
 		<child link="camera_link" />
-		<origin xyz="${0.03} ${0} 0.005" rpy="0 0.1 0" />
-		<axis xyz="0 0 1" />
+		<origin xyz="${0} ${0.06} 0.005" rpy="0 0.1 ${3.14/2}" />
+		<axis xyz="0 0 1" />
+	</joint>
+<!-- ======================================================== -->
+	<!-- Define joint between camera and frame -->
+	<joint name="joint_imu_frame" type="fixed">
+		<parent link="plate1" />
+		<child link="imu_link" />
+		<origin xyz="0 0 0" rpy="0 0 0" />
 	</joint>
 <!-- ======================================================== -->

Commit message: URDF: Cleaned up Kwad model naming, added comments

File: urdf/Kwad.xacro (robot description, xacro)
@@ -2,11 +2,17 @@
 <robot xmlns:xacro="http://www.ros.org/wiki/xacro" name="Kwad">
 <!-- ======================================================== -->
+	<!-- Constants -->
+	<xacro:property name="pi_value" value="3.14159263" />
+	<!-- Dimensions for cross beam arms -->
 	<xacro:property name="width" value="0.0315" />
 	<xacro:property name="length" value="0.45" />
 	<xacro:property name="height" value="0.01" />
+	<!-- Mass of cross beam arms -->
 	<xacro:property name="mass_fr" value="0.5" />
+	<!-- Dimension of propellors -->
+	<xacro:property name="radiusp" value="0.20" />
+	<!-- Mass of propellors -->
 	<xacro:property name="mass_pr" value="0.0055" />
-	<xacro:property name="pi_value" value="3.14159263" />
-	<xacro:property name="radiusp" value="0.20" />
+	<!-- Location of propellors -->
 	<xacro:property name="prop_loc" value="0.15909" />
 <!-- ======================================================== -->
@@ -24,4 +30,7 @@
 	</xacro:macro>
 <!-- ======================================================== -->
+	<!-- Base link -->
+	<link name="base_link"/>
+<!-- ======================================================== -->
 	<link name="arm_1">
 		<visual>
@@ -58,6 +67,4 @@
 	</link>
 <!-- ======================================================== -->
-	<link name="base_link"/>
-<!-- ======================================================== -->
 	<link name="plate1">
 		<visual>
@@ -77,5 +84,5 @@
 	</link>
 <!-- ======================================================== -->
-	<link name="cyl1">
+	<link name="cyl_fr">
 		<visual>
 			<origin xyz="0 0 0" rpy="0 0 0" />
@@ -94,5 +101,5 @@
 	</link>
 <!-- ======================================================== -->
-	<link name="cyl2">
+	<link name="cyl_bl">
 		<visual>
 			<origin xyz="0 0 0" rpy="0 0 0" />
@@ -111,5 +118,5 @@
 	</link>
 <!-- ======================================================== -->
-	<link name="cyl3">
+	<link name="cyl_fl">
 		<visual>
 			<origin xyz="0 0 0" rpy="0 0 0" />
@@ -128,5 +135,5 @@
 	</link>
 <!-- ======================================================== -->
-	<link name="cyl4">
+	<link name="cyl_br">
 		<visual>
 			<origin xyz="0 0 0" rpy="0 0 0" />
@@ -298,32 +305,32 @@
 	</joint>
 <!-- ======================================================== -->
-<!-- Define joint between cyl1 and frame -->
-	<joint name="joint_cyl1_frame" type="fixed">
-		<parent link="arm_2" />
-		<child link="cyl1" />
+<!-- Define joint between cyl_fr and frame -->
+	<joint name="joint_cyl_fr_frame" type="fixed">
+		<parent link="arm_2" />
+		<child link="cyl_fr" />
 		<origin xyz="${prop_loc - 0.01} ${prop_loc - 0.01} 0.01" rpy="0 0 0" />
 		<axis xyz="0 0 1" />
 	</joint>
 <!-- ======================================================== -->
-<!-- Define joint between cyl2 and frame -->
-	<joint name="joint_cyl2_frame" type="fixed">
-		<parent link="arm_2" />
-		<child link="cyl2" />
+<!-- Define joint between cyl_bl and frame -->
+	<joint name="joint_cyl_bl_frame" type="fixed">
+		<parent link="arm_2" />
+		<child link="cyl_bl" />
 		<origin xyz="${-prop_loc + 0.01} ${-prop_loc + 0.01} 0.01" rpy="0 0 0" />
 		<axis xyz="0 0 1" />
 	</joint>
 <!-- ======================================================== -->
-<!-- Define joint between cyl3 and frame -->
-	<joint name="joint_cyl3_frame" type="fixed">
-		<parent link="arm_1" />
-		<child link="cyl3" />
+<!-- Define joint between cyl_fl and frame -->
+	<joint name="joint_cyl_fl_frame" type="fixed">
+		<parent link="arm_1" />
+		<child link="cyl_fl" />
 		<origin xyz="${-prop_loc + 0.01} ${prop_loc - 0.01} 0.01" rpy="0 0 0" />
 		<axis xyz="0 0 1" />
 	</joint>
 <!-- ======================================================== -->
-<!-- Define joint between cyl4 and frame -->
-	<joint name="joint_cyl4_frame" type="fixed">
-		<parent link="arm_1" />
-		<child link="cyl4" />
+<!-- Define joint between cyl_br and frame -->
+	<joint name="joint_cyl_br_frame" type="fixed">
+		<parent link="arm_1" />
+		<child link="cyl_br" />
 		<origin xyz="${prop_loc - 0.01} ${-prop_loc + 0.01} 0.01" rpy="0 0 0" />
 		<axis xyz="0 0 1" />
