Commit message: URDF: Fixed inertia of quad model, cleaned up urdf files

File: urdf/Kwad.xacro (robot description, xacro)
@@ -1,4 +1,8 @@
 <?xml version="1.0"?>
 <robot xmlns:xacro="http://www.ros.org/wiki/xacro" name="Kwad">
+<!-- ======================================================== -->
+	<xacro:include filename="$(find robotuna_ekf_simulator)/urdf/material.xacro" />
+	<xacro:include filename="$(find robotuna_ekf_simulator)/urdf/macros.xacro"/>
+	<xacro:include filename="$(find robotuna_ekf_simulator)/urdf/Kwad.gazebo" />
 <!-- ======================================================== -->
 	<!-- Constants -->
@@ -7,249 +11,134 @@
 	<xacro:property name="width" value="0.0315" />
 	<xacro:property name="length" value="0.45" />
-	<xacro:property name="height" value="0.01" />
+	<xacro:property name="height" value="0.015" />
 	<!-- Mass of cross beam arms -->
-	<xacro:property name="mass_fr" value="0.5" />
-	<!-- Dimension of propellors -->
+	<xacro:property name="mass_fr" value="0.8" />
+	<!-- Dimension of propellers -->
 	<xacro:property name="radiusp" value="0.20" />
-	<!-- Mass of propellors -->
+	<!-- Mass of propellers -->
 	<xacro:property name="mass_pr" value="0.0055" />
-	<!-- Location of propellors -->
+	<!-- Location of propellers -->
 	<xacro:property name="prop_loc" value="0.15909" />
 <!-- ======================================================== -->
-	<xacro:include filename="$(find robotuna_ekf_simulator)/urdf/material.xacro" />
-	<xacro:include filename="$(find robotuna_ekf_simulator)/urdf/Kwad.gazebo" />
-<!-- ======================================================== -->
-	<!-- Define inertial macro -->
-	<xacro:macro name="default_inertial" params="mass p ix_value iy_value iz_value" >
-		<inertial>
-			<origin xyz="0 0 0" rpy="0 0 ${p}" />
-			<mass value="${mass}" />
-			<inertia ixx="${ix_value}" ixy="0" ixz="0"
-					 iyy="${iy_value}" iyz="0" izz="${iz_value}" />
-		</inertial>
-	</xacro:macro>
-<!-- ======================================================== -->
+<!-- ======================================================== -->
+<!-- ####################### -->
+		<!-- Links -->
+<!-- ####################### -->
 	<!-- Base link -->
 	<link name="base_link"/>
 <!-- ======================================================== -->
-	<link name="arm_1">
-		<visual>
-			<origin xyz="0 0 0" rpy="0 0 ${pi_value/4}" />
-			<geometry>
-				<box size="${width} ${length} ${height}" />
-			</geometry>
-			<material name="red" />
-		</visual>
-		<collision>
-			<origin xyz="0 0 0" rpy="0 0 ${pi_value/4}" />
-			<geometry>
-				<box size="${width} ${length} ${height}" />
-			</geometry>
-		</collision>
-		<xacro:default_inertial mass="${mass_fr}" p="${pi_value/4}" ix_value="${0.04989/2}" iy_value="${0.04989/2}" iz_value="${0.24057/2}" />
-	</link>
-<!-- ======================================================== -->
-	<link name="arm_2">
-		<visual>
-			<origin xyz="0 0 0" rpy="0 0 ${-pi_value/4}" />
-			<geometry>
-				<box size="${width} ${length} ${height}" />
-			</geometry>
-			<material name="white" />
-		</visual>
-		<collision>
-			<origin xyz="0 0 0" rpy="0 0 ${-pi_value/4}" />
-			<geometry>
-				<box size="${width} ${length} ${height}" />
-			</geometry>
-		</collision>
-		<xacro:default_inertial mass="${mass_fr}" p="${-pi_value/4}" ix_value="${0.04989/2}" iy_value="${0.04989/2}" iz_value="${0.24057/2}" />
-	</link>
-<!-- ======================================================== -->
-	<link name="plate1">
-		<visual>
-			<origin xyz="0 0 0" rpy="0 0 0" />
-			<geometry>
-				<box size="${0.12} ${0.12} ${0.01}" />
-			</geometry>
-			<material name="black" />
-		</visual>
-		<collision>
-			<origin xyz="0 0 0" rpy="0 0 0" />
-			<geometry>
-				<box size="${0.12} ${0.12} ${0.01}" />
-			</geometry>
-		</collision>
-		<xacro:default_inertial mass="${0.01}" p="${0}" ix_value="${0}" iy_value="${0}" iz_value="${2.4-5}" />
-	</link>
-<!-- ======================================================== -->
-	<link name="cyl_fr">
-		<visual>
-			<origin xyz="0 0 0" rpy="0 0 0" />
-			<geometry>
-				<cylinder radius="0.016" length="0.02" />
-			</geometry>
-			<material name="golden" />
-		</visual>
-		<collision>
-			<origin xyz="0 0 0" rpy="0 0 0" />
-			<geometry>
-				<cylinder radius="0.016" length="0.02" />
-			</geometry>
-		</collision>
-		<xacro:default_inertial mass="${0.01}" p="${0}" ix_value="${8.95e-6}" iy_value="${8.95e-6}" iz_value="${2.23e-4}" />
-	</link>
-<!-- ======================================================== -->
-	<link name="cyl_bl">
-		<visual>
-			<origin xyz="0 0 0" rpy="0 0 0" />
-			<geometry>
-				<cylinder radius="0.016" length="0.02" />
-			</geometry>
-			<material name="golden" />
-		</visual>
-		<collision>
-			<origin xyz="0 0 0" rpy="0 0 0" />
-			<geometry>
-				<cylinder radius="0.016" length="0.02" />
-			</geometry>
-		</collision>
-		<xacro:default_inertial mass="${0.01}" p="${0}" ix_value="${8.95e-6}" iy_value="${8.95e-6}" iz_value="${2.23e-4}" />
-	</link>
-<!-- ======================================================== -->
-	<link name="cyl_fl">
-		<visual>
-			<origin xyz="0 0 0" rpy="0 0 0" />
-			<geometry>
-				<cylinder radius="0.016" length="0.02" />
-			</geometry>
-			<material name="golden" />
-		</visual>
-		<collision>
-			<origin xyz="0 0 0" rpy="0 0 0" />
-			<geometry>
-				<cylinder radius="0.016" length="0.02" />
-			</geometry>
-		</collision>
-		<xacro:default_inertial mass="${0.01}" p="${0}" ix_value="${8.95e-6}" iy_value="${8.95e-6}" iz_value="${2.23e-4}" />
-	</link>
-<!-- ======================================================== -->
-	<link name="cyl_br">
-		<visual>
-			<origin xyz="0 0 0" rpy="0 0 0" />
-			<geometry>
-				<cylinder radius="0.016" length="0.02" />
-			</geometry>
-			<material name="golden" />
-		</visual>
-		<collision>
-			<origin xyz="0 0 0" rpy="0 0 0" />
-			<geometry>
-				<cylinder radius="0.016" length="0.02" />
-			</geometry>
-		</collision>
-		<xacro:default_inertial mass="${0.01}" p="${0}" ix_value="${8.95e-6}" iy_value="${8.95e-6}" iz_value="${2.23e-4}" />
-	</link>
-<!-- ======================================================== -->
-	<link name="camera_link">
-		<visual>
-			<origin xyz="0 0 0" rpy="0 0 0" />
-			<geometry>
-				<box size="0.01 0.01 0.01" />
-			</geometry>
-			<material name="red" />
-		</visual>
-		<collision>
-			<origin xyz="0 0 0" rpy="0 0 0" />
-			<geometry>
-				<box size="0.01 0.01 0.01" />
-			</geometry>
-		</collision>
-		<xacro:default_inertial mass="${1e-5}" p="${0}" ix_value="${1e-6}" iy_value="${1e-6}" iz_value="${1e-6}" />
-	</link>
-<!-- ======================================================== -->
-	<link name="imu_link">
-		<visual>
-			<origin xyz="0 0 0" rpy="0 0 0" />
-			<geometry>
-				<box size="0.01 0.01 0.01" />
-			</geometry>
-			<material name="red" />
-		</visual>
-		<collision>
-			<origin xyz="0 0 0" rpy="0 0 0" />
-			<geometry>
-				<box size="0.01 0.01 0.01" />
-			</geometry>
-		</collision>
-		<xacro:default_inertial mass="${1e-5}" p="${0}" ix_value="${1e-6}" iy_value="${1e-6}" iz_value="${1e-6}" />
-	</link>
-<!-- ======================================================== -->
+<!-- Quadcopter frame links -->
+	<!-- First arm -->
+	<xacro:boxLink
+		name="arm_1"
+		mass="${mass_fr}"
+		x_dim="${width}" y_dim="${length}" z_dim="${height}"
+		y="${pi_value/4}"
+		color="red"
+	/>
+	<!-- Second arm -->
+	<xacro:boxLink
+		name="arm_2"
+		mass="${mass_fr}"
+		x_dim="${width}" y_dim="${length}" z_dim="${height}"
+		y="${-pi_value/4}"
+		color="white"
+	/>
+	<!-- Electronics mounting plate -->
+	<xacro:boxLink
+		name="plate1"
+		mass="0.01"
+		x_dim="0.12" y_dim="0.12" z_dim="0.01"
+		color="black"
+	/>
+<!-- ======================================================== -->
+<!-- Motor links -->
+	<!-- Front right motor -->
+	<xacro:cylinderLink
+		name="cyl_fr"
+		mass="0.01"
+		radius="0.016"
+		height="0.02"
+		color="golden"
+	/>
+	<!-- Back left motor -->
+	<xacro:cylinderLink
+		name="cyl_bl"
+		mass="0.01"
+		radius="0.016"
+		height="0.02"
+		color="golden"
+	/>
+	<!-- Front left motor -->
+	<xacro:cylinderLink
+		name="cyl_fl"
+		mass="0.01"
+		radius="0.016"
+		height="0.02"
+		color="golden"
+	/>
+	<!-- Back right motor -->
+	<xacro:cylinderLink
+		name="cyl_br"
+		mass="0.01"
+		radius="0.016"
+		height="0.02"
+		color="golden"
+	/>
+<!-- ======================================================== -->
+<!-- Propeller links -->
 	<!-- Propellers of the quad: fr, fl, br, bl -->
-	<link name="prop_front_right">
-		<visual>
-			<origin xyz="0 0 0" rpy="0 0 0" />
-			<geometry>
-				<box size="${0.03302/3} ${radiusp*0.8} ${0.001}" />
-			</geometry>
-			<material name="black" />
-		</visual>
-		<collision>
-			<origin xyz="0 0 0" rpy="0 0 0" />
-			<geometry>
-				<box size="${0.03302/3} ${radiusp*0.8} ${0.001}" />
-			</geometry>
-		</collision>
-		<xacro:default_inertial mass="${mass_pr}" p="${0}" ix_value="${0}" iy_value="${0}" iz_value="${4.42448e-5}" />
-	</link>
-	<link name="prop_front_left">
-		<visual>
-			<origin xyz="0 0 0" rpy="0 0 0" />
-			<geometry>
-				<box size="${0.03302/3} ${radiusp*0.8} ${0.001}" />
-			</geometry>
-			<material name="black"/>
-		</visual>
-		<collision>
-			<origin xyz="0 0 0" rpy="0 0 0" />
-			<geometry>
-				<box size="${0.03302/3} ${radiusp*0.8} ${0.001}" />
-			</geometry>
-		</collision>
-		<xacro:default_inertial mass="${mass_pr}" p="${0}"  ix_value="${0}" iy_value="${0}" iz_value="${4.42448e-5}" />
-	</link>
-	<link name="prop_back_right">
-		<visual>
-			<origin xyz="0 0 0" rpy="0 0 0" />
-			<geometry>
-				<box size="${0.03302/3} ${radiusp*0.8} ${0.001}" />
-			</geometry>
-			<material name="black"/>
-		</visual>
-		<collision>
-			<origin xyz="0 0 0" rpy="0 0 0" />
-			<geometry>
-				<box size="${0.03302/3} ${radiusp*0.8} ${0.001}" />
-			</geometry>
-		</collision>
-		<xacro:default_inertial mass="${mass_pr}" p="${0}"  ix_value="${0}" iy_value="${0}" iz_value="${4.42448e-5}" />
-	</link>
-	<link name="prop_back_left">
-		<visual>
-			<origin xyz="0 0 0" rpy="0 0 0" />
-			<geometry>
-				<box size="${0.03302/3} ${radiusp*0.8} ${0.001}" />
-			</geometry>
-			<material name="black"/>
-		</visual>
-		<collision>
-			<origin xyz="0 0 0" rpy="0 0 0" />
-			<geometry>
-				<box size="${0.03302/3} ${radiusp*0.8} ${0.001}" />
-			</geometry>
-		</collision>
-		<xacro:default_inertial mass="${mass_pr}" p="${0}"  ix_value="${0}" iy_value="${0}" iz_value="${4.42448e-5}" />
-	</link>
-<!-- ======================================================== -->
+	<!-- For the propellers we don't use the boxLink macros, because we need to make their
+		 inertials "flat" (no inertia around x or y axis). Thus we construct them the
+		 traditional way. -->
+	<xacro:boxLink_customInertia
+		name="prop_front_right"
+		mass="${mass_pr}"
+		x_dim="${0.03302/3}" y_dim="${radiusp*0.8}" z_dim="0.005"
+		ix="0" iy="0" iz="${4.42448e-5}"
+		color="black"
+	/>
+	<xacro:boxLink_customInertia
+		name="prop_front_left"
+		mass="${mass_pr}"
+		x_dim="${0.03302/3}" y_dim="${radiusp*0.8}" z_dim="0.005"
+		ix="0" iy="0" iz="${4.42448e-5}"
+		color="black"
+	/>
+	<xacro:boxLink_customInertia
+		name="prop_back_right"
+		mass="${mass_pr}"
+		x_dim="${0.03302/3}" y_dim="${radiusp*0.8}" z_dim="0.005"
+		ix="0" iy="0" iz="${4.42448e-5}"
+		color="black"
+	/>
+	<xacro:boxLink_customInertia
+		name="prop_back_left"
+		mass="${mass_pr}"
+		x_dim="${0.03302/3}" y_dim="${radiusp*0.8}" z_dim="0.005"
+		ix="0" iy="0" iz="${4.42448e-5}"
+		color="black"
+	/>
+<!-- ======================================================== -->
+<!-- Sensor links -->
+	<!-- Camera -->
+	<xacro:boxLink
+		name="camera_link"
+		mass="${1e-5}"
+		x_dim="0.01" y_dim="0.01" z_dim="0.01"
+		color="red"
+	/>
+	<!-- IMU -->
+	<xacro:boxLink
+		name="imu_link"
+		mass="${1e-5}"
+		x_dim="0.01" y_dim="0.01" z_dim="0.01"
+		color="red"
+	/>
+<!-- ======================================================== -->
+<!-- ======================================================== -->
+<!-- ####################### -->
+		<!-- Joints -->
+<!-- ####################### -->
 	<joint name="base_joint" type="fixed">
 		<parent link="base_link" />
@@ -352,4 +241,8 @@
 	</joint>
 <!-- ======================================================== -->
+<!-- ======================================================== -->
+<!-- ####################### -->
+	<!-- Transmissions -->
+<!-- ####################### -->
 <!-- Add transmission elements -->
 	<transmission name="front_right_motor_joint" >

File: urdf/material.xacro (robot description, xacro)
@@ -1,4 +1,4 @@
 <?xml version="1.0"?>
-<robot>
+<robot xmlns:xacro="http://www.ros.org/wiki/xacro">
 	<material name="white">
 		<color rgba="0.8 0.8 0.8 1" />

Commit message: URDF: Rotated Kwad model such that X=front, Y=left, Z=up to match roll-pitch-yaw. Formerly X=right, Y=front, Z=up.

File: urdf/Kwad.xacro (robot description, xacro)
@@ -153,73 +153,68 @@
 		<axis xyz="0 0 1" />
 	</joint>
-<!-- ======================================================== -->
+	<!-- Define joint between plate1 and frame -->
+	<joint name="joint_plate1_frame" type="fixed">
+		<parent link="arm_2" />
+		<child link="plate1" />
+		<origin xyz="${0} ${0} 0.005" rpy="0 0 0" />
+		<axis xyz="0 0 1" />
+	</joint>
+<!-- ======================================================== -->
+<!-- Propeller joints -->
 	<!-- Define joint between prop fr and frame -->
+	<joint name="joint_front_left_prop" type="continuous">
+		<parent link="arm_2" />
+		<child link="prop_front_left" />
+		<origin xyz="${prop_loc - 0.01} ${prop_loc - 0.01} 0.021" rpy="0 0 0"/>
+		<axis xyz="0 0 1" />
+	</joint>
+	<!-- Define joint between prop fl and frame -->
+	<joint name="joint_back_left_prop" type="continuous">
+		<parent link="arm_1" />
+		<child link="prop_back_left" />
+		<origin xyz="${-prop_loc + 0.01} ${prop_loc - 0.01} 0.021" rpy="0 0 0" />
+		<axis xyz="0 0 1" />
+	</joint>
+<!-- Define joint between prop br and frame -->
 	<joint name="joint_front_right_prop" type="continuous">
-		<parent link="arm_2" />
+		<parent link="arm_1" />
 		<child link="prop_front_right" />
-		<origin xyz="${prop_loc - 0.01} ${prop_loc - 0.01} 0.021" rpy="0 0 0"/>
-		<axis xyz="0 0 1" />
-	</joint>
-<!-- ======================================================== -->
-	<!-- Define joint between prop fl and frame -->
-	<joint name="joint_front_left_prop" type="continuous">
-		<parent link="arm_1" />
-		<child link="prop_front_left" />
-		<origin xyz="${-prop_loc + 0.01} ${prop_loc - 0.01} 0.021" rpy="0 0 0" />
-		<axis xyz="0 0 1" />
-	</joint>
-<!-- ======================================================== -->
+		<origin xyz="${prop_loc - 0.01} ${-prop_loc + 0.01} 0.021" rpy="0 0 0" />
+		<axis xyz="0 0 1" />
+	</joint>
 <!-- Define joint between prop br and frame -->
 	<joint name="joint_back_right_prop" type="continuous">
-		<parent link="arm_1" />
+		<parent link="arm_2" />
 		<child link="prop_back_right" />
-		<origin xyz="${prop_loc - 0.01} ${-prop_loc + 0.01} 0.021" rpy="0 0 0" />
-		<axis xyz="0 0 1" />
-	</joint>
-<!-- ======================================================== -->
-<!-- Define joint between prop br and frame -->
-	<joint name="joint_back_left_prop" type="continuous">
-		<parent link="arm_2" />
-		<child link="prop_back_left" />
 		<origin xyz="${-prop_loc + 0.01} ${-prop_loc + 0.01} 0.021" rpy="0 0 0" />
 		<axis xyz="0 0 1" />
 	</joint>
 <!-- ======================================================== -->
-<!-- Define joint between plate1 and frame -->
-	<joint name="joint_plate1_frame" type="fixed">
-		<parent link="arm_2" />
-		<child link="plate1" />
-		<origin xyz="${0} ${0} 0.005" rpy="0 0 0" />
-		<axis xyz="0 0 1" />
-	</joint>
-<!-- ======================================================== -->
+<!-- Motor cylinder joints -->
 <!-- Define joint between cyl_fr and frame -->
+	<joint name="joint_cyl_fl_frame" type="fixed">
+		<parent link="arm_2" />
+		<child link="cyl_fl" />
+		<origin xyz="${prop_loc - 0.01} ${prop_loc - 0.01} 0.01" rpy="0 0 0" />
+		<axis xyz="0 0 1" />
+	</joint>
+<!-- Define joint between cyl_bl and frame -->
+	<joint name="joint_cyl_br_frame" type="fixed">
+		<parent link="arm_2" />
+		<child link="cyl_br" />
+		<origin xyz="${-prop_loc + 0.01} ${-prop_loc + 0.01} 0.01" rpy="0 0 0" />
+		<axis xyz="0 0 1" />
+	</joint>
+<!-- Define joint between cyl_fl and frame -->
+	<joint name="joint_cyl_bl_frame" type="fixed">
+		<parent link="arm_1" />
+		<child link="cyl_bl" />
+		<origin xyz="${-prop_loc + 0.01} ${prop_loc - 0.01} 0.01" rpy="0 0 0" />
+		<axis xyz="0 0 1" />
+	</joint>
+<!-- Define joint between cyl_br and frame -->
 	<joint name="joint_cyl_fr_frame" type="fixed">
-		<parent link="arm_2" />
+		<parent link="arm_1" />
 		<child link="cyl_fr" />
-		<origin xyz="${prop_loc - 0.01} ${prop_loc - 0.01} 0.01" rpy="0 0 0" />
-		<axis xyz="0 0 1" />
-	</joint>
-<!-- ======================================================== -->
-<!-- Define joint between cyl_bl and frame -->
-	<joint name="joint_cyl_bl_frame" type="fixed">
-		<parent link="arm_2" />
-		<child link="cyl_bl" />
-		<origin xyz="${-prop_loc + 0.01} ${-prop_loc + 0.01} 0.01" rpy="0 0 0" />
-		<axis xyz="0 0 1" />
-	</joint>
-<!-- ======================================================== -->
-<!-- Define joint between cyl_fl and frame -->
-	<joint name="joint_cyl_fl_frame" type="fixed">
-		<parent link="arm_1" />
-		<child link="cyl_fl" />
-		<origin xyz="${-prop_loc + 0.01} ${prop_loc - 0.01} 0.01" rpy="0 0 0" />
-		<axis xyz="0 0 1" />
-	</joint>
-<!-- ======================================================== -->
-<!-- Define joint between cyl_br and frame -->
-	<joint name="joint_cyl_br_frame" type="fixed">
-		<parent link="arm_1" />
-		<child link="cyl_br" />
 		<origin xyz="${prop_loc - 0.01} ${-prop_loc + 0.01} 0.01" rpy="0 0 0" />
 		<axis xyz="0 0 1" />
@@ -230,5 +225,5 @@
 		<parent link="plate1" />
 		<child link="camera_link" />
-		<origin xyz="${0} ${0.06} 0.005" rpy="0 0.1 ${3.14/2}" />
+		<origin xyz="0.06 0 0.005" rpy="0 0.1 0" />
 		<axis xyz="0 0 1" />
 	</joint>
